Commit message: added core URDF

File: description/robot_core.xacro (robot description, xacro)
@@ -1,4 +1,5 @@
 <?xml version="1.0"?>
 <robot xmlns:xacro="http://www.ros.org/wiki/xacro">
+    <xacro:include filename="inertial_macros.xacro"/>
     <material name="white">
         <color rgba="1 1 1 1"/>
@@ -26,8 +27,19 @@
             <origin xyz="0.15 0 0.075"/>
             <geometry>
+<!--                <cylinder radius="0.15" length="0.15"/> -->
                 <box size="0.3 0.3 0.15"/>
             </geometry>
             <material name="white"/>
         </visual>
+        <collision>
+            <origin xyz="0.15 0 0.075"/>
+            <geometry>
+<!--                <cylinder radius="0.15" length="0.15"/> -->
+                <box size="0.3 0.3 0.15"/>
+            </geometry>
+        </collision>
+        <xacro:inertial_box mass="0.5" x="0.3" y="0.3" z="0.15">
+            <origin xyz="0.15 0 0.075" rpy="0 0 0 "/>
+        </xacro:inertial_box>
     </link>
     <!-- LEFT WHEEL -->
@@ -45,4 +57,12 @@
             <material name="blue"/>
         </visual>
+        <collision>
+            <geometry>
+                <cylinder radius="0.05" length="0.04"/>
+            </geometry>
+        </collision>
+        <xacro:inertial_cylinder mass="0.1" length="0.04" radius="0.05">
+            <origin xyz="0 0 0" rpy="0 0 0"/>
+        </xacro:inertial_cylinder>
     </link>
     <!-- RIGHT WHEEL -->
@@ -60,4 +80,34 @@
             <material name="blue"/>
         </visual>
+        <collision>
+            <geometry>
+                <cylinder radius="0.05" length="0.04"/>
+            </geometry>
+        </collision>
+        <xacro:inertial_cylinder mass="0.1" length="0.04" radius="0.05">
+            <origin xyz="0 0 0" rpy="0 0 0"/>
+        </xacro:inertial_cylinder>
+    </link>
+    <!-- CASTOR WHEEL LINK -->
+    <joint name="caster_wheel_joint" type="fixed">
+        <parent link="chassis"/>
+        <child link="caster_wheel"/>
+        <origin xyz="0.24 0 0"/>
+    </joint>
+    <link name="caster_wheel">
+        <visual>
+            <geometry>
+                <sphere radius="0.05"/>
+            </geometry>
+            <material name="blue"/>
+        </visual>
+        <collision>
+            <geometry>
+                <sphere radius="0.05"/>
+            </geometry>
+        </collision>
+        <xacro:inertial_sphere mass="0.1" radius="0.05">
+            <origin xyz="0 0 0" rpy="0 0 0"/>
+        </xacro:inertial_sphere>
     </link>
 </robot>

Commit message: cylinder chassis

File: description/robot_core.xacro (robot description, xacro)
@@ -27,6 +27,6 @@
             <origin xyz="0.15 0 0.075"/>
             <geometry>
-<!--                <cylinder radius="0.15" length="0.15"/> -->
-                <box size="0.3 0.3 0.15"/>
+                <cylinder radius="0.175" length="0.070"/>
+<!--                <box size="0.3 0.3 0.15"/>  -->
             </geometry>
             <material name="white"/>
@@ -35,11 +35,11 @@
             <origin xyz="0.15 0 0.075"/>
             <geometry>
-<!--                <cylinder radius="0.15" length="0.15"/> -->
-                <box size="0.3 0.3 0.15"/>
+                <cylinder radius="0.175" length="0.070"/>
+<!--                <box size="0.3 0.3 0.15"/>   -->
             </geometry>
         </collision>
-        <xacro:inertial_box mass="0.5" x="0.3" y="0.3" z="0.15">
-            <origin xyz="0.15 0 0.075" rpy="0 0 0 "/>
-        </xacro:inertial_box>
+        <xacro:inertial_cylinder mass="0.5" radius="0.175" length="0.070">
+            <origin xyz="0.175 0 0.070" rpy="0 0 0 "/>
+        </xacro:inertial_cylinder>
     </link>
     <gazebo reference="chassis">
@@ -50,5 +50,5 @@
         <parent link="base_link"/>
         <child link="left_wheel"/>
-        <origin xyz="0 0.175 0" rpy="-${pi/2} 0 0" />
+        <origin xyz="0 0.125 0.025" rpy="-${pi/2} 0 0" />
         <axis xyz="0 0 1"/>
     </joint>
@@ -76,5 +76,5 @@
         <parent link="base_link"/>
         <child link="right_wheel"/>
-        <origin xyz="0 -0.175 0" rpy="${pi/2} 0 0" />
+        <origin xyz="0 -0.125 0.025" rpy="${pi/2} 0 0" />
         <axis xyz="0 0 -1"/>
     </joint>
@@ -102,5 +102,5 @@
         <parent link="chassis"/>
         <child link="caster_wheel"/>
-        <origin xyz="0.24 0 0"/>
+        <origin xyz="0.24 0 0.025"/>
     </joint>
     <link name="caster_wheel">

Commit message: modded joystick scale for cmd_vel

File: description/robot_core.xacro (robot description, xacro)
@@ -56,5 +56,5 @@
         <visual>
             <geometry>
-                <cylinder radius="0.05" length="0.04"/>
+                <cylinder radius="0.036" length="0.04"/>
             </geometry>
             <material name="blue"/>
@@ -62,8 +62,8 @@
         <collision>
             <geometry>
-                <cylinder radius="0.05" length="0.04"/>
+                <cylinder radius="0.036" length="0.04"/>
             </geometry>
         </collision>
-        <xacro:inertial_cylinder mass="0.1" length="0.04" radius="0.05">
+        <xacro:inertial_cylinder mass="0.1" length="0.04" radius="0.036">
             <origin xyz="0 0 0" rpy="0 0 0"/>
         </xacro:inertial_cylinder>
@@ -82,5 +82,5 @@
         <visual>
             <geometry>
-                <cylinder radius="0.05" length="0.04"/>
+                <cylinder radius="0.036" length="0.04"/>
             </geometry>
             <material name="blue"/>
@@ -88,8 +88,8 @@
         <collision>
             <geometry>
-                <cylinder radius="0.05" length="0.04"/>
+                <cylinder radius="0.036" length="0.04"/>
             </geometry>
         </collision>
-        <xacro:inertial_cylinder mass="0.1" length="0.04" radius="0.05">
+        <xacro:inertial_cylinder mass="0.1" length="0.04" radius="0.036">
             <origin xyz="0 0 0" rpy="0 0 0"/>
         </xacro:inertial_cylinder>
@@ -107,5 +107,5 @@
         <visual>
             <geometry>
-                <sphere radius="0.05"/>
+                <sphere radius="0.036"/>
             </geometry>
             <material name="blue"/>
@@ -113,8 +113,8 @@
         <collision>
             <geometry>
-                <sphere radius="0.05"/>
+                <sphere radius="0.036"/>
             </geometry>
         </collision>
-        <xacro:inertial_sphere mass="0.1" radius="0.05">
+        <xacro:inertial_sphere mass="0.1" radius="0.036">
             <origin xyz="0 0 0" rpy="0 0 0"/>
         </xacro:inertial_sphere>
